Commit message: Misc

File: Packages/alex_description/urdf/JointWorkaround.urdf.xacro (robot description, xacro)
@@ -40,4 +40,19 @@
     </visual>
   </link>
+  <link name="link1">
+    <visual>
+      <geometry>
+        <cylinder length="${l1}" radius="0.003"/>
+      </geometry>
+      <origin rpy="0 ${pi/2} 0" xyz="${l1/2} 0 0"/>
+      <material name="blue"/>
+    </visual>
+  </link>
+  <joint name="base_to_link1" type="continuous">
+    <parent link="base_link"/>
+    <child link="link1"/>
+    <axis rpy="0 0 0" xyz="0 0 1"/>
+    <origin rpy="0 0 ${pi/4}" xyz="0 0 0"/>
+  </joint>
   <link name="link2">
     <visual>
@@ -54,4 +69,19 @@
     <axis rpy="0 0 0" xyz="0 0 1"/>
     <origin rpy="0 0 ${3 * pi/4}" xyz="0 0 0"/>
+  </joint>
+  <link name="link3">
+    <visual>
+      <geometry>
+        <cylinder length="${l3}" radius="0.003"/>
+      </geometry>
+      <origin rpy="0 ${pi/2} 0" xyz="${l3/2} 0 0"/>
+      <material name="red"/>
+    </visual>
+  </link>
+  <joint name="link1_to_link3" type="continuous">
+    <parent link="link1"/>
+    <child link="link3"/>
+    <axis rpy="0 0 0" xyz="0 0 1"/>
+    <origin rpy="0 0 ${pi/2}" xyz="${l1} 0 0"/>
   </joint>
   <link name="link4">
@@ -79,5 +109,5 @@
     </visual>
   </link>
-  <joint name="link4_to_link5" type="fixed">
+  <joint name="link4_to_link5" type="continuous">
     <parent link="link4"/>
     <child link="link5"/>

Commit message: misc

File: Packages/alex_description/urdf/JointWorkaround.urdf.xacro (robot description, xacro)
@@ -100,3 +100,33 @@
     <origin rpy="0 0 0" xyz="${l5} 0 0"/>
   </joint>
+  <link name="link1">
+    <visual>
+      <geometry>
+        <cylinder length="${l1}" radius="0.003"/>
+      </geometry>
+      <origin rpy="0 ${pi/2} 0" xyz="${l1/2} 0 0"/>
+      <material name="red"/>
+    </visual>
+  </link>
+  <joint name="base_to_link1" type="continuous">
+    <parent link="base_link"/>
+    <child link="link1"/>
+    <axis rpy="0 0 0" xyz="0 0 1"/>
+    <origin rpy="0 0 ${pi/4}" xyz="0 0 0"/>
+  </joint>
+  <link name="link3">
+    <visual>
+      <geometry>
+        <cylinder length="${l3}" radius="0.003"/>
+      </geometry>
+      <origin rpy="0 ${pi/2} 0" xyz="${l3/2} 0 0"/>
+      <material name="red"/>
+    </visual>
+  </link>
+  <joint name="link1_to_link3" type="continuous">
+    <parent link="link1"/>
+    <child link="link3"/>
+    <axis rpy="0 0 0" xyz="0 0 1"/>
+    <origin rpy="0 0 ${pi/2}" xyz="${l1} 0 0"/>
+  </joint>
 </robot>

Commit message: Before test day

File: Packages/alex_description/urdf/JointWorkaround.urdf.xacro (robot description, xacro)
@@ -130,36 +130,3 @@
     <origin rpy="0 0 0" xyz="${l5} 0 0"/>
   </joint>
-<<<<<<< HEAD
-  <link name="link1">
-    <visual>
-      <geometry>
-        <cylinder length="${l1}" radius="0.003"/>
-      </geometry>
-      <origin rpy="0 ${pi/2} 0" xyz="${l1/2} 0 0"/>
-      <material name="red"/>
-    </visual>
-  </link>
-  <joint name="base_to_link1" type="continuous">
-    <parent link="base_link"/>
-    <child link="link1"/>
-    <axis rpy="0 0 0" xyz="0 0 1"/>
-    <origin rpy="0 0 ${pi/4}" xyz="0 0 0"/>
-  </joint>
-  <link name="link3">
-    <visual>
-      <geometry>
-        <cylinder length="${l3}" radius="0.003"/>
-      </geometry>
-      <origin rpy="0 ${pi/2} 0" xyz="${l3/2} 0 0"/>
-      <material name="red"/>
-    </visual>
-  </link>
-  <joint name="link1_to_link3" type="continuous">
-    <parent link="link1"/>
-    <child link="link3"/>
-    <axis rpy="0 0 0" xyz="0 0 1"/>
-    <origin rpy="0 0 ${pi/2}" xyz="${l1} 0 0"/>
-  </joint>
-=======
->>>>>>> 22a4a1888f98473f5509272baba5a561a8260483
 </robot>
