Commit message: Full leg fkine

File: Packages/alex_description/urdf/FullBody.urdf.xacro (robot description, xacro)
@@ -1,4 +1,23 @@
 <?xml version="1.0"?>
 <robot name="ALEX" xmlns:xacro="http://ros.org/wiki/xacro">
+  <xacro:property name="base_offset_x" value="0" />
+  <xacro:property name="base_offset_y" value="-0.5" />
+  <xacro:property name="base_offset_z" value="-0.1" />
+  <xacro:property name="hip_offset_x" value="0.1" />
+  <xacro:property name="hip_offset_y" value="0.1" />
+  <xacro:property name="hip_offset_z" value="0.1" />
+  <xacro:property name="hip_length" value="0" />
+  <xacro:property name="knee_length_a" value="0.1" />
+  <xacro:property name="knee_length_b" value="0.3" />
+  <xacro:property name="shin_length_a" value="0.309" />
+  <xacro:property name="shin_length_b" value="0.305" />
+  <xacro:property name="shin_connection_length" value="0.115" />
+  <xacro:property name="ankle_a_offset" value="0.07475" />
+  <xacro:property name="ankle_length_b" value="0.02735" />
+  <xacro:property name="ankle_length_c" value="0.0432" />
+  <xacro:property name="ankle_length_d1" value="0.1493" />
+  <xacro:property name="ankle_length_d2" value="0.155795" />
+  <xacro:property name="foot_length_a" value="0.055" />
+  <xacro:property name="foot_length_b" value="0.055" />
   <xacro:property name="l1" value="0.1" />
   <xacro:property name="l2" value="0.3" />
@@ -13,5 +32,4 @@
   <xacro:property name="l10" value="0.04025" />
   <xacro:property name="l11" value="0.07475" />
-  <xacro:property name="theta1" value="0.7853981625" />
   <material name="red">
     <color rgba="1 0 0 1"/>
@@ -35,4 +53,185 @@
     <color rgba="1 1 1 1"/>
   </material>
+  <xacro:macro name="leg" params="prefix reflect">
+    <link name="${prefix}_hip_link">
+      <visual>
+        <geometry>
+          <cylinder length="${knee_length_a}" radius="0.003"/>
+        </geometry>
+      </visual>
+    </link>
+    <joint name="base_link_to_${prefix}_hip_link" type="continuous">
+      <parent link="base_link"/>
+      <child link="${prefix}_hip_link"/>
+      <axis rpy="0 0 0" xyz="0 0 1"/>
+      <origin rpy="0 ${pi/2} ${pi}" xyz="${base_offset_x} ${reflect * base_offset_y} ${base_offset_z}"/>
+    </joint>
+    <link name="${prefix}_knee_link_b">
+      <visual>
+        <geometry>
+          <cylinder length="${knee_length_b}" radius="0.003"/>
+        </geometry>
+        <origin rpy="0 ${pi/2} 0" xyz="${knee_length_b/2} 0 0"/>
+        <material name="blue"/>
+      </visual>
+    </link>
+    <joint name="${prefix}_hip_link_to_knee_link_b" type="continuous">
+      <parent link="${prefix}_hip_link"/>
+      <child link="${prefix}_knee_link_b"/>
+      <axis rpy="0 0 0" xyz="0 0 1"/>
+      <origin rpy="${pi/2} ${-pi/4} 0" xyz="${hip_offset_x} ${reflect * hip_offset_y} ${hip_offset_z}"/>
+    </joint>
+    <link name="${prefix}_shin_link_b">
+      <visual>
+        <geometry>
+          <cylinder length="${shin_length_b}" radius="0.003"/>
+        </geometry>
+        <origin rpy="0 ${pi/2} 0" xyz="${shin_length_b/2} 0 0"/>
+        <material name="blue"/>
+      </visual>
+    </link>
+    <joint name="${prefix}_knee_link_b_to_${prefix}_shin_link_b" type="continuous">
+      <parent link="${prefix}_knee_link_b"/>
+      <child link="${prefix}_shin_link_b"/>
+      <axis rpy="0 0 0" xyz="0 0 1"/>
+      <origin rpy="0 0 ${-pi/2}" xyz="${knee_length_b} 0 0"/>
+    </joint>
+    <link name="${prefix}_knee_link_a">
+      <visual>
+        <geometry>
+          <cylinder length="${knee_length_a}" radius="0.003"/>
+        </geometry>
+        <origin rpy="0 ${pi/2} 0" xyz="${knee_length_a/2} 0 0"/>
+        <material name="blue"/>
+      </visual>
+    </link>
+    <joint name="${prefix}_knee_link_b_to_${prefix}_knee_link_a" type="continuous">
+      <parent link="${prefix}_knee_link_b"/>
+      <child link="${prefix}_knee_link_a"/>
+      <axis rpy="0 0 0" xyz="0 0 1"/>
+      <origin rpy="0 0 ${-pi/2}" xyz="0 0 0"/>
+    </joint>
+    <link name="${prefix}_shin_link_a">
+      <visual>
+        <geometry>
+          <cylinder length="${shin_length_a}" radius="0.003"/>
+        </geometry>
+        <origin rpy="0 ${pi/2} 0" xyz="${shin_length_a/2} 0 0"/>
+        <material name="blue"/>
+      </visual>
+    </link>
+    <joint name="${prefix}_knee_link_a_to_${prefix}_shin_link_a" type="continuous">
+      <parent link="${prefix}_knee_link_a"/>
+      <child link="${prefix}_shin_link_a"/>
+      <axis rpy="0 0 0" xyz="0 0 1"/>
+      <origin rpy="0 0 ${pi/2}" xyz="${knee_length_a} 0 0"/>
+    </joint>
+    <link name="${prefix}_shin_link_connection">
+      <visual>
+        <geometry>
+          <cylinder length="0" radius="0.003"/>
+        </geometry>
+        <origin rpy="0 ${pi/2} 0" xyz="${shin_connection_length/2} 0 0"/>
+        <material name="blue"/>
+      </visual>
+    </link>
+    <joint name="${prefix}_shink_link_b_to_${prefix}_shin_link_connection" type="continuous">
+      <parent link="${prefix}_shin_link_b"/>
+      <child link="${prefix}_shin_link_connection"/>
+      <axis rpy="0 0 0" xyz="0 0 1"/>
+      <origin rpy="0 0 0" xyz="${shin_connection_length} 0 0"/>
+    </joint>
+    <link name="${prefix}_foot_link_b">
+      <visual>
+        <geometry>
+          <cylinder length="${foot_length_b}" radius="0.003"/>
+        </geometry>
+        <origin rpy="0 ${pi/2} 0" xyz="${foot_length_b/2} 0 0"/>
+        <material name="blue"/>
+      </visual>
+    </link>
+    <joint name="${prefix}_shin_link_connection_to_${prefix}_foot_link_b" type="continuous">
+      <parent link="${prefix}_shin_link_connection"/>
+      <child link="${prefix}_foot_link_b"/>
+      <axis rpy="0 0 0" xyz="0 0 1"/>
+      <origin rpy="0 0 ${-pi/2}" xyz="${shin_length_a - shin_connection_length} 0 0"/>
+    </joint>
+    <link name="${prefix}_ankle_link_a">
+      <visual>
+        <geometry>
+          <cylinder length="${ankle_length_b}" radius="0.003"/>
+        </geometry>
+        <origin rpy="0 ${pi/2} 0" xyz="${ankle_length_b/2} 0 0"/>
+        <material name="blue"/>
+      </visual>
+    </link>
+    <joint name="${prefix}_shin_link_b_to_${prefix}_ankle_link_a" type="continuous">
+      <parent link="${prefix}_shin_link_b"/>
+      <child link="${prefix}_ankle_link_a"/>
+      <axis rpy="0 0 0" xyz="0 0 1"/>
+      <origin rpy="0 0 ${pi/2}" xyz="${ankle_a_offset} 0 0"/>
+    </joint>
+    <link name="${prefix}_ankle_link_b">
+      <visual>
+        <geometry>
+          <cylinder length="${ankle_length_c}" radius="0.003"/>
+        </geometry>
+        <origin rpy="0 ${pi/2} 0" xyz="${ankle_length_c/2} 0 0"/>
+        <material name="blue"/>
+      </visual>
+    </link>
+    <joint name="${prefix}_ankle_link_a_to_${prefix}_ankle_link_b" type="continuous">
+      <parent link="${prefix}_ankle_link_a"/>
+      <child link="${prefix}_ankle_link_b"/>
+      <axis rpy="0 0 0" xyz="0 0 1"/>
+      <origin rpy="0 0 ${-pi/8}" xyz="${ankle_length_b} 0 0"/>
+    </joint>
+    <link name="${prefix}_ankle_link_c_1">
+      <visual>
+        <geometry>
+          <cylinder length="${ankle_length_d1}" radius="0.003"/>
+        </geometry>
+        <origin rpy="0 ${pi/2} 0" xyz="${ankle_length_d1/2} 0 0"/>
+        <material name="blue"/>
+      </visual>
+    </link>
+    <joint name="${prefix}_ankle_link_b_to_${prefix}_ankle_link_c_1" type="continuous">
+      <parent link="${prefix}_ankle_link_b"/>
+      <child link="${prefix}_ankle_link_c_1"/>
+      <axis rpy="0 0 0" xyz="0 0 1"/>
+      <origin rpy="0 0 ${-pi/4}" xyz="${ankle_length_c} 0 0"/>
+    </joint>
+    <link name="${prefix}_ankle_link_c_2">
+      <visual>
+        <geometry>
+          <cylinder length="${ankle_length_d2}" radius="0.003"/>
+        </geometry>
+        <origin rpy="0 ${pi/2} 0" xyz="${ankle_length_d2/2} 0 0"/>
+        <material name="blue"/>
+      </visual>
+    </link>
+    <joint name="${prefix}_ankle_link_c_1_to_${prefix}_ankle_link_c_2" type="prismatic">
+      <limit lower="${-0.0515/2}" upper="${0.0515/2}" effort="1" velocity="1"/>
+      <parent link="${prefix}_ankle_link_c_1"/>
+      <child link="${prefix}_ankle_link_c_2"/>
+      <axis rpy="0 0 0" xyz="1 0 0"/>
+      <origin rpy="0 0 0" xyz="${0.0515/2} 0 0"/>
+    </joint>
+    <link name="${prefix}_foot_link_a">
+      <visual>
+        <geometry>
+          <cylinder length="${foot_length_a}" radius="0.003"/>
+        </geometry>
+        <origin rpy="0 ${pi/2} 0" xyz="${foot_length_a/2} 0 0"/>
+        <material name="blue"/>
+      </visual>
+    </link>
+    <joint name="${prefix}_ankle_link_c_2_to_${prefix}_foot_link_a" type="continuous">
+      <parent link="${prefix}_ankle_link_c_2"/>
+      <child link="${prefix}_foot_link_a"/>
+      <axis rpy="0 0 0" xyz="0 0 1"/>
+      <origin rpy="0 0 ${-pi/2}" xyz="${ankle_length_d2} 0 0"/>
+    </joint>
+  </xacro:macro>
   <link name="base_link">
     <visual>
@@ -40,93 +239,5 @@
     </visual>
   </link>
-  <link name="link1">
-    <visual>
-      <geometry>
-        <cylinder length="${l1}" radius="0.003"/>
-      </geometry>
-      <origin rpy="0 ${pi/2} 0" xyz="${l1/2} 0 0"/>
-      <material name="blue"/>
-    </visual>
-  </link>
-  <joint name="base_to_link1" type="continuous">
-    <parent link="base_link"/>
-    <child link="link1"/>
-    <axis rpy="0 0 0" xyz="0 0 1"/>
-    <origin rpy="0 0 ${pi/4}" xyz="0 0 0"/>
-  </joint>
-  <link name="link2">
-    <visual>
-      <geometry>
-        <cylinder length="${l2}" radius="0.003"/>
-      </geometry>
-      <origin rpy="0 ${pi/2} 0" xyz="${l2/2} 0 0"/>
-      <material name="blue"/>
-    </visual>
-  </link>
-  <joint name="base_to_link2" type="continuous">
-    <parent link="base_link"/>
-    <child link="link2"/>
-    <axis rpy="0 0 0" xyz="0 0 1"/>
-    <origin rpy="0 0 ${3 * pi/4}" xyz="0 0 0"/>
-  </joint>
-  <link name="link3">
-    <visual>
-      <geometry>
-        <cylinder length="${l3}" radius="0.003"/>
-      </geometry>
-      <origin rpy="0 ${pi/2} 0" xyz="${l3/2} 0 0"/>
-      <material name="red"/>
-    </visual>
-  </link>
-  <joint name="link1_to_link3" type="continuous">
-    <parent link="link1"/>
-    <child link="link3"/>
-    <axis rpy="0 0 0" xyz="0 0 1"/>
-    <origin rpy="0 0 ${pi/2}" xyz="${l1} 0 0"/>
-  </joint>
-  <link name="link4">
-    <visual>
-      <geometry>
-        <cylinder length="${l4}" radius="0.003"/>
-      </geometry>
-      <origin rpy="0 ${pi/2} 0" xyz="${l4/2} 0 0"/>
-      <material name="red"/>
-    </visual>
-  </link>
-  <joint name="link2_to_link4" type="continuous">
-    <parent link="link2"/>
-    <child link="link4"/>
-    <axis rpy="0 0 0" xyz="0 0 1"/>
-    <origin rpy="0 0 ${-pi/2}" xyz="${l2} 0 0"/>
-  </joint>
-  <link name="link5">
-    <visual>
-      <geometry>
-        <cylinder length="${l5}" radius="0.003"/>
-      </geometry>
-      <origin rpy="0 ${pi/2} 0" xyz="${l5/2} 0 0"/>
-      <material name="red"/>
-    </visual>
-  </link>
-  <joint name="link4_to_link5" type="continuous">
-    <parent link="link4"/>
-    <child link="link5"/>
-    <axis rpy="0 0 0" xyz="0 0 1"/>
-    <origin rpy="0 0 0" xyz="${l4} 0 0"/>
-  </joint>
-  <link name="null">
-    <visual>
-      <geometry>
-        <cylinder length="0" radius="0.003"/>
-      </geometry>
-      <origin rpy="0 ${pi/2} 0" xyz="0 0 0"/>
-      <material name="red"/>
-    </visual>
-  </link>
-  <joint name="link5_to_null" type="continuous">
-    <parent link="link5"/>
-    <child link="null"/>
-    <axis rpy="0 0 0" xyz="0 0 1"/>
-    <origin rpy="0 0 0" xyz="${l5} 0 0"/>
-  </joint>
+  <xacro:leg prefix="right" reflect="1" />
+  <xacro:leg prefix="left" reflect="-1" />
 </robot>

Commit message: ikine progress

File: Packages/alex_description/urdf/FullBody.urdf.xacro (robot description, xacro)
@@ -235,7 +235,4 @@
   </xacro:macro>
   <link name="base_link">
-    <visual>
-      <material name="yellow"/>
-    </visual>
   </link>
   <xacro:leg prefix="right" reflect="1" />

Commit message: ikine

File: Packages/alex_description/urdf/FullBody.urdf.xacro (robot description, xacro)
@@ -1,35 +1,22 @@
 <?xml version="1.0"?>
 <robot name="ALEX" xmlns:xacro="http://ros.org/wiki/xacro">
-  <xacro:property name="base_offset_x" value="0" />
-  <xacro:property name="base_offset_y" value="-0.5" />
-  <xacro:property name="base_offset_z" value="-0.1" />
-  <xacro:property name="hip_offset_x" value="0.1" />
-  <xacro:property name="hip_offset_y" value="0.1" />
-  <xacro:property name="hip_offset_z" value="0.1" />
-  <xacro:property name="hip_length" value="0" />
-  <xacro:property name="knee_length_a" value="0.1" />
-  <xacro:property name="knee_length_b" value="0.3" />
-  <xacro:property name="shin_length_a" value="0.309" />
-  <xacro:property name="shin_length_b" value="0.305" />
-  <xacro:property name="shin_connection_length" value="0.115" />
-  <xacro:property name="ankle_a_offset" value="0.07475" />
-  <xacro:property name="ankle_length_b" value="0.02735" />
-  <xacro:property name="ankle_length_c" value="0.0432" />
-  <xacro:property name="ankle_length_d1" value="0.1493" />
-  <xacro:property name="ankle_length_d2" value="0.155795" />
-  <xacro:property name="foot_length_a" value="0.055" />
-  <xacro:property name="foot_length_b" value="0.055" />
-  <xacro:property name="l1" value="0.1" />
-  <xacro:property name="l2" value="0.3" />
-  <xacro:property name="l3" value="0.309" />
-  <xacro:property name="l4" value="0.115" />
-  <xacro:property name="l5" value="0.19" />
-  <xacro:property name="l6" value="0.02735" />
-  <xacro:property name="l7" value="0.0432" />
-  <xacro:property name="l8_a" value="0.1493" />
-  <xacro:property name="l8_b" value="0.155795" />
-  <xacro:property name="l9" value="0.055" />
-  <xacro:property name="l10" value="0.04025" />
-  <xacro:property name="l11" value="0.07475" />
+  <xacro:property name="o_base_to_hip_x" value="0" />
+  <xacro:property name="o_base_to_hip_y" value="-0.5" />
+  <xacro:property name="o_base_to_hip_z" value="-0.1" />
+  <xacro:property name="o_hip_to_knee_x" value="0.1" />
+  <xacro:property name="o_hip_to_knee_y" value="0.1" />
+  <xacro:property name="o_hip_to_knee_z" value="0.1" />
+  <xacro:property name="l_knee_a" value="0.1" />
+  <xacro:property name="l_knee_b" value="0.3" />
+  <xacro:property name="l_shin_a" value="0.309" />
+  <xacro:property name="l_shin_b" value="0.305" />
+  <xacro:property name="l_shin_connection" value="0.115" />
+  <xacro:property name="l_ankle_connection" value="0.07475" />
+  <xacro:property name="l_ankle_a" value="0.02735" />
+  <xacro:property name="l_ankle_b" value="0.0432" />
+  <xacro:property name="l_ankle_c1" value="0.1493" />
+  <xacro:property name="l_ankle_c2" value="0.155795" />
+  <xacro:property name="l_foot_a" value="0.055" />
+  <xacro:property name="l_foot_b" value="0.055" />
   <material name="red">
     <color rgba="1 0 0 1"/>
@@ -55,9 +42,4 @@
   <xacro:macro name="leg" params="prefix reflect">
     <link name="${prefix}_hip_link">
-      <visual>
-        <geometry>
-          <cylinder length="${knee_length_a}" radius="0.003"/>
-        </geometry>
-      </visual>
     </link>
     <joint name="base_link_to_${prefix}_hip_link" type="continuous">
@@ -65,12 +47,12 @@
       <child link="${prefix}_hip_link"/>
       <axis rpy="0 0 0" xyz="0 0 1"/>
-      <origin rpy="0 ${pi/2} ${pi}" xyz="${base_offset_x} ${reflect * base_offset_y} ${base_offset_z}"/>
+      <origin rpy="0 ${pi/2} ${pi}" xyz="${o_base_to_hip_x} ${reflect * o_base_to_hip_y} ${o_base_to_hip_z}"/>
     </joint>
     <link name="${prefix}_knee_link_b">
       <visual>
         <geometry>
-          <cylinder length="${knee_length_b}" radius="0.003"/>
-        </geometry>
-        <origin rpy="0 ${pi/2} 0" xyz="${knee_length_b/2} 0 0"/>
+          <cylinder length="${l_knee_b}" radius="0.003"/>
+        </geometry>
+        <origin rpy="0 ${pi/2} 0" xyz="${l_knee_b/2} 0 0"/>
         <material name="blue"/>
       </visual>
@@ -80,12 +62,12 @@
       <child link="${prefix}_knee_link_b"/>
       <axis rpy="0 0 0" xyz="0 0 1"/>
-      <origin rpy="${pi/2} ${-pi/4} 0" xyz="${hip_offset_x} ${reflect * hip_offset_y} ${hip_offset_z}"/>
+      <origin rpy="${pi/2} ${-pi/4} 0" xyz="${o_hip_to_knee_x} ${reflect * o_hip_to_knee_y} ${o_hip_to_knee_z}"/>
     </joint>
     <link name="${prefix}_shin_link_b">
       <visual>
         <geometry>
-          <cylinder length="${shin_length_b}" radius="0.003"/>
-        </geometry>
-        <origin rpy="0 ${pi/2} 0" xyz="${shin_length_b/2} 0 0"/>
+          <cylinder length="${l_shin_b}" radius="0.003"/>
+        </geometry>
+        <origin rpy="0 ${pi/2} 0" xyz="${l_shin_b/2} 0 0"/>
         <material name="blue"/>
       </visual>
@@ -95,12 +77,12 @@
       <child link="${prefix}_shin_link_b"/>
       <axis rpy="0 0 0" xyz="0 0 1"/>
-      <origin rpy="0 0 ${-pi/2}" xyz="${knee_length_b} 0 0"/>
+      <origin rpy="0 0 ${-pi/2}" xyz="${l_knee_b} 0 0"/>
     </joint>
     <link name="${prefix}_knee_link_a">
       <visual>
         <geometry>
-          <cylinder length="${knee_length_a}" radius="0.003"/>
-        </geometry>
-        <origin rpy="0 ${pi/2} 0" xyz="${knee_length_a/2} 0 0"/>
+          <cylinder length="${l_knee_a}" radius="0.003"/>
+        </geometry>
+        <origin rpy="0 ${pi/2} 0" xyz="${l_knee_a/2} 0 0"/>
         <material name="blue"/>
       </visual>
@@ -115,7 +97,7 @@
       <visual>
         <geometry>
-          <cylinder length="${shin_length_a}" radius="0.003"/>
-        </geometry>
-        <origin rpy="0 ${pi/2} 0" xyz="${shin_length_a/2} 0 0"/>
+          <cylinder length="${l_shin_a}" radius="0.003"/>
+        </geometry>
+        <origin rpy="0 ${pi/2} 0" xyz="${l_shin_a/2} 0 0"/>
         <material name="blue"/>
       </visual>
@@ -125,5 +107,5 @@
       <child link="${prefix}_shin_link_a"/>
       <axis rpy="0 0 0" xyz="0 0 1"/>
-      <origin rpy="0 0 ${pi/2}" xyz="${knee_length_a} 0 0"/>
+      <origin rpy="0 0 ${pi/2}" xyz="${l_knee_a} 0 0"/>
     </joint>
     <link name="${prefix}_shin_link_connection">
@@ -132,5 +114,5 @@
           <cylinder length="0" radius="0.003"/>
         </geometry>
-        <origin rpy="0 ${pi/2} 0" xyz="${shin_connection_length/2} 0 0"/>
+        <origin rpy="0 ${pi/2} 0" xyz="${l_shin_connection/2} 0 0"/>
         <material name="blue"/>
       </visual>
@@ -140,12 +122,12 @@
       <child link="${prefix}_shin_link_connection"/>
       <axis rpy="0 0 0" xyz="0 0 1"/>
-      <origin rpy="0 0 0" xyz="${shin_connection_length} 0 0"/>
+      <origin rpy="0 0 0" xyz="${l_shin_connection} 0 0"/>
     </joint>
     <link name="${prefix}_foot_link_b">
       <visual>
         <geometry>
-          <cylinder length="${foot_length_b}" radius="0.003"/>
-        </geometry>
-        <origin rpy="0 ${pi/2} 0" xyz="${foot_length_b/2} 0 0"/>
+          <cylinder length="${l_foot_b}" radius="0.003"/>
+        </geometry>
+        <origin rpy="0 ${pi/2} 0" xyz="${l_foot_b/2} 0 0"/>
         <material name="blue"/>
       </visual>
@@ -155,12 +137,12 @@
       <child link="${prefix}_foot_link_b"/>
       <axis rpy="0 0 0" xyz="0 0 1"/>
-      <origin rpy="0 0 ${-pi/2}" xyz="${shin_length_a - shin_connection_length} 0 0"/>
+      <origin rpy="0 0 ${-pi/2}" xyz="${l_shin_a - l_shin_connection} 0 0"/>
     </joint>
     <link name="${prefix}_ankle_link_a">
       <visual>
         <geometry>
-          <cylinder length="${ankle_length_b}" radius="0.003"/>
-        </geometry>
-        <origin rpy="0 ${pi/2} 0" xyz="${ankle_length_b/2} 0 0"/>
+          <cylinder length="${l_ankle_a}" radius="0.003"/>
+        </geometry>
+        <origin rpy="0 ${pi/2} 0" xyz="${l_ankle_a/2} 0 0"/>
         <material name="blue"/>
       </visual>
@@ -170,12 +152,12 @@
       <child link="${prefix}_ankle_link_a"/>
       <axis rpy="0 0 0" xyz="0 0 1"/>
-      <origin rpy="0 0 ${pi/2}" xyz="${ankle_a_offset} 0 0"/>
+      <origin rpy="0 0 ${pi/2}" xyz="${l_ankle_connection} 0 0"/>
     </joint>
     <link name="${prefix}_ankle_link_b">
       <visual>
         <geometry>
-          <cylinder length="${ankle_length_c}" radius="0.003"/>
-        </geometry>
-        <origin rpy="0 ${pi/2} 0" xyz="${ankle_length_c/2} 0 0"/>
+          <cylinder length="${l_ankle_b}" radius="0.003"/>
+        </geometry>
+        <origin rpy="0 ${pi/2} 0" xyz="${l_ankle_b/2} 0 0"/>
         <material name="blue"/>
       </visual>
@@ -185,12 +167,12 @@
       <child link="${prefix}_ankle_link_b"/>
       <axis rpy="0 0 0" xyz="0 0 1"/>
-      <origin rpy="0 0 ${-pi/8}" xyz="${ankle_length_b} 0 0"/>
+      <origin rpy="0 0 ${-pi/8}" xyz="${l_ankle_a} 0 0"/>
     </joint>
     <link name="${prefix}_ankle_link_c_1">
       <visual>
         <geometry>
-          <cylinder length="${ankle_length_d1}" radius="0.003"/>
-        </geometry>
-        <origin rpy="0 ${pi/2} 0" xyz="${ankle_length_d1/2} 0 0"/>
+          <cylinder length="${l_ankle_c1}" radius="0.003"/>
+        </geometry>
+        <origin rpy="0 ${pi/2} 0" xyz="${l_ankle_c1/2} 0 0"/>
         <material name="blue"/>
       </visual>
@@ -200,12 +182,12 @@
       <child link="${prefix}_ankle_link_c_1"/>
       <axis rpy="0 0 0" xyz="0 0 1"/>
-      <origin rpy="0 0 ${-pi/4}" xyz="${ankle_length_c} 0 0"/>
+      <origin rpy="0 0 ${-pi/4}" xyz="${l_ankle_b} 0 0"/>
     </joint>
     <link name="${prefix}_ankle_link_c_2">
       <visual>
         <geometry>
-          <cylinder length="${ankle_length_d2}" radius="0.003"/>
-        </geometry>
-        <origin rpy="0 ${pi/2} 0" xyz="${ankle_length_d2/2} 0 0"/>
+          <cylinder length="${l_ankle_c2}" radius="0.003"/>
+        </geometry>
+        <origin rpy="0 ${pi/2} 0" xyz="${l_ankle_c2/2} 0 0"/>
         <material name="blue"/>
       </visual>
@@ -221,7 +203,7 @@
       <visual>
         <geometry>
-          <cylinder length="${foot_length_a}" radius="0.003"/>
-        </geometry>
-        <origin rpy="0 ${pi/2} 0" xyz="${foot_length_a/2} 0 0"/>
+          <cylinder length="${l_foot_a}" radius="0.003"/>
+        </geometry>
+        <origin rpy="0 ${pi/2} 0" xyz="${l_foot_a/2} 0 0"/>
         <material name="blue"/>
       </visual>
@@ -231,5 +213,5 @@
       <child link="${prefix}_foot_link_a"/>
       <axis rpy="0 0 0" xyz="0 0 1"/>
-      <origin rpy="0 0 ${-pi/2}" xyz="${ankle_length_d2} 0 0"/>
+      <origin rpy="0 0 ${-pi/2}" xyz="${l_ankle_c2} 0 0"/>
     </joint>
   </xacro:macro>

Commit message: Moving kinematics

File: Packages/alex_description/urdf/FullBody.urdf.xacro (robot description, xacro)
@@ -58,5 +58,5 @@
       </visual>
     </link>
-    <joint name="${prefix}_hip_link_to_knee_link_b" type="continuous">
+    <joint name="${prefix}_hip_link_to_${prefix}_knee_link_b" type="continuous">
       <parent link="${prefix}_hip_link"/>
       <child link="${prefix}_knee_link_b"/>
